Commit message: Add 2D LiDAR sensor to mobile robot model

File: src/mobile_robot_description/urdf/mobile_robot.urdf.xacro (robot description, xacro)
@@ -14,14 +14,10 @@
     <visual>
       <origin xyz="0 0 0.08" rpy="0 0 0"/>
-      <geometry>
-        <box size="0.30 0.22 0.10"/>
-      </geometry>
+      <geometry><box size="0.30 0.22 0.10"/></geometry>
       <material name="blue"/>
     </visual>
     <collision>
       <origin xyz="0 0 0.08" rpy="0 0 0"/>
-      <geometry>
-        <box size="0.30 0.22 0.10"/>
-      </geometry>
+      <geometry><box size="0.30 0.22 0.10"/></geometry>
     </collision>
     <inertial>
@@ -41,14 +37,10 @@
       <visual>
         <origin xyz="0 0 0" rpy="1.57079632679 0 0"/>
-        <geometry>
-          <cylinder radius="0.05" length="0.025"/>
-        </geometry>
+        <geometry><cylinder radius="0.05" length="0.025"/></geometry>
         <material name="dark_grey"/>
       </visual>
       <collision>
         <origin xyz="0 0 0" rpy="1.57079632679 0 0"/>
-        <geometry>
-          <cylinder radius="0.05" length="0.025"/>
-        </geometry>
+        <geometry><cylinder radius="0.05" length="0.025"/></geometry>
       </collision>
       <inertial>
@@ -68,15 +60,6 @@
   <xacro:wheel name="right_wheel" y="-0.1225"/>
   <link name="caster_wheel">
-    <visual>
-      <geometry>
-        <sphere radius="0.025"/>
-      </geometry>
-      <material name="black"/>
-    </visual>
-    <collision>
-      <geometry>
-        <sphere radius="0.025"/>
-      </geometry>
-    </collision>
+    <visual><geometry><sphere radius="0.025"/></geometry><material name="black"/></visual>
+    <collision><geometry><sphere radius="0.025"/></geometry></collision>
     <inertial>
       <mass value="0.05"/>
@@ -90,4 +73,47 @@
     <origin xyz="-0.11 0 0.025" rpy="0 0 0"/>
   </joint>
+  <!-- 2D LiDAR frame and Gazebo Sim sensor -->
+  <link name="lidar_link">
+    <visual>
+      <geometry><cylinder radius="0.035" length="0.035"/></geometry>
+      <material name="black"/>
+    </visual>
+    <collision>
+      <geometry><cylinder radius="0.035" length="0.035"/></geometry>
+    </collision>
+    <inertial>
+      <mass value="0.12"/>
+      <inertia ixx="0.0001" ixy="0.0" ixz="0.0"
+               iyy="0.0001" iyz="0.0" izz="0.0001"/>
+    </inertial>
+  </link>
+  <joint name="lidar_joint" type="fixed">
+    <parent link="base_link"/>
+    <child link="lidar_link"/>
+    <origin xyz="0.02 0 0.17" rpy="0 0 0"/>
+  </joint>
+  <gazebo reference="lidar_link">
+    <sensor name="front_lidar" type="gpu_lidar">
+      <topic>/scan</topic>
+      <update_rate>10</update_rate>
+      <lidar>
+        <scan>
+          <horizontal>
+            <samples>360</samples>
+            <resolution>1</resolution>
+            <min_angle>-3.14159</min_angle>
+            <max_angle>3.14159</max_angle>
+          </horizontal>
+        </scan>
+        <range>
+          <min>0.12</min>
+          <max>8.0</max>
+          <resolution>0.01</resolution>
+        </range>
+      </lidar>
+      <always_on>true</always_on>
+      <visualize>true</visualize>
+    </sensor>
+  </gazebo>
   <!-- Gazebo Sim Harmonic differential-drive controller -->
   <gazebo>
